File: MOSFET/MOSFET.brd (EAGLE design)
At the start: 120 x 120 mm, 10 parts

Commit message: 4mm Aufbohren !
Parts:
- GND, IN0, IN1, OUT0, OUT1, VS: value 9774100982 -> M4 x 10mm; device Wurth_Assembly_WA-SMST:WA-SMST_9774100982 -> Wurth_Assembly_WA-SMSI:WA-SMSI_9774100482
