File: MOSFET/MOSFET.sch (EAGLE design)
At the start: 10 parts

Commit message: 4mm Aufbohren !
Parts:
- GND, IN0, IN1, OUT0, OUT1, VS: value 9774100982 -> M4 x 10mm; device Wurth_Assembly_WA-SMST:WA-SMST_9774XXX982_9774100982 -> Wurth_Assembly_WA-SMSI:WA-SMSI_9774XXX482_9774100482
Other:
- note added: "M4 Aufbohren auf 4mm für Bananenstecker !"
Changed lines of the file:
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@@
 <drawing>
 <settings>
-<setting alwaysvectorfont="yes"/>
+<setting alwaysvectorfont="no"/>
 <setting verticaltext="up"/>
 </settings>
@@
 <part name="GND21" library="supply1" library_urn="urn:adsk.eagle:library:371" deviceset="GND" device=""/>
 <part name="C1" library="Wurth_Elektronik_Passive_Capacitors_rev19a" library_urn="urn:adsk.eagle:library:491551" deviceset="WCAP-CSGP_0402" device="" package3d_urn="urn:adsk.eagle:package:491821/3" technology="_885012205037" value="100n"/>
-<part name="IN0" library="Wurth_Assembly_WA-SMST" library_urn="urn:adsk.eagle:library:14418621" deviceset="WA-SMST_9774XXX982" device="_9774100982" package3d_urn="urn:adsk.eagle:package:14328907/2" value=" 9774100982 "/>
-<part name="IN1" library="Wurth_Assembly_WA-SMST" library_urn="urn:adsk.eagle:library:14418621" deviceset="WA-SMST_9774XXX982" device="_9774100982" package3d_urn="urn:adsk.eagle:package:14328907/2" value=" 9774100982 "/>
-<part name="GND" library="Wurth_Assembly_WA-SMST" library_urn="urn:adsk.eagle:library:14418621" deviceset="WA-SMST_9774XXX982" device="_9774100982" package3d_urn="urn:adsk.eagle:package:14328907/2" value=" 9774100982 "/>
-<part name="OUT1" library="Wurth_Assembly_WA-SMST" library_urn="urn:adsk.eagle:library:14418621" deviceset="WA-SMST_9774XXX982" device="_9774100982" package3d_urn="urn:adsk.eagle:package:14328907/2" value=" 9774100982 "/>
-<part name="OUT0" library="Wurth_Assembly_WA-SMST" library_urn="urn:adsk.eagle:library:14418621" deviceset="WA-SMST_9774XXX982" device="_9774100982" package3d_urn="urn:adsk.eagle:package:14328907/2" value=" 9774100982 "/>
-<part name="VS" library="Wurth_Assembly_WA-SMST" library_urn="urn:adsk.eagle:library:14418621" deviceset="WA-SMST_9774XXX982" device="_9774100982" package3d_urn="urn:adsk.eagle:package:14328907/2" value=" 9774100982 "/>
+<part name="IN0" library="Wurth_Assembly_WA-SMSI" library_urn="urn:adsk.eagle:library:14418591" deviceset="WA-SMSI_9774XXX482" device="_9774100482" package3d_urn="urn:adsk.eagle:package:14321898/2" value="M4 x 10mm"/>
+<part name="IN1" library="Wurth_Assembly_WA-SMSI" library_urn="urn:adsk.eagle:library:14418591" deviceset="WA-SMSI_9774XXX482" device="_9774100482" package3d_urn="urn:adsk.eagle:package:14321898/2" value="M4 x 10mm"/>
+<part name="GND" library="Wurth_Assembly_WA-SMSI" library_urn="urn:adsk.eagle:library:14418591" deviceset="WA-SMSI_9774XXX482" device="_9774100482" package3d_urn="urn:adsk.eagle:package:14321898/2" value="M4 x 10mm"/>
+<part name="OUT1" library="Wurth_Assembly_WA-SMSI" library_urn="urn:adsk.eagle:library:14418591" deviceset="WA-SMSI_9774XXX482" device="_9774100482" package3d_urn="urn:adsk.eagle:package:14321898/2" value="M4 x 10mm"/>
+<part name="OUT0" library="Wurth_Assembly_WA-SMSI" library_urn="urn:adsk.eagle:library:14418591" deviceset="WA-SMSI_9774XXX482" device="_9774100482" package3d_urn="urn:adsk.eagle:package:14321898/2" value="M4 x 10mm"/>
+<part name="VS" library="Wurth_Assembly_WA-SMSI" library_urn="urn:adsk.eagle:library:14418591" deviceset="WA-SMSI_9774XXX482" device="_9774100482" package3d_urn="urn:adsk.eagle:package:14321898/2" value="M4 x 10mm"/>
 </parts>
 <sheets>
 <sheet>
 <plain>
+<text x="71.12" y="0" size="1.778" layer="91">M4 Aufbohren auf 4mm für Bananenstecker !</text>
 </plain>
 <instances>
